File: Qwiic-OpenLog.brd (EAGLE design)
At the start: 25.4 x 26.7 mm, 49 parts, among them J1 MICRO-SD, J2 SMD, J3 PTH, J4 SMD, J5 ISP, Q1 16MHZ, U2 ATMEGA328P

Commit message: Add files via upload
Parts:
- removed U$18: (no value), buzzard_labels (14):OPENLOG0
- C1: value 4.7uF -> 4.7 uF 10V; device SparkFun-Capacitors:0603 -> SeekOps_capacitors:C0805
- moved R1 1.27 mm to (17.8, 20.3)
Routing:
- net N$3: track 1.28 -> 2.55 mm
- net N$4: track 4.39 -> 3.49 mm
Other:
- board text added: "new text added here"
