File: Qwiic-OpenLog.sch (EAGLE design)
At the start: 31 parts, among them J1 MICRO-SD, J2 SMD, J3 PTH, J4 SMD, J5 ISP, Q1 16MHZ, U2 ATMEGA328P

Commit message: Add files via upload
Parts:
- C1: value 4.7uF -> 4.7 uF 10V; device SparkFun-Capacitors:4.7UF-0603-6.3V-(10%) -> SeekOps_capacitors:C0805C475J8RACAUTO
Other:
- moved on the sheet: C2
